File: BottomBoard.sch (KiCad schematic (older format))
At the start: 19 parts, among them IC2 A3916GESTR-T, IC3 A3916GESTR-T, J4 Conn_01x06_Female, J5 Conn_01x06_Female, J6 Conn_01x08_Female

Commit message: routed and reshaped
Parts:
- removed C7, C8: CP, Capacitor_SMD:CP_Elec_3x5.3, symbol Device:CP
- added C15, C8: C, Capacitor_SMD:C_0805_2012Metric, symbol Device:C
- added C20, C21: C, Capacitor_SMD:C_0402_1005Metric, symbol Device:C
- added D1, D2: LED, LED_SMD:LED_0603_1608Metric, symbol Device:LED
- added JP1: Jumper_NO_Small, Jumper:SolderJumper-2_P1.3mm_Open_Pad1.0x1.5mm, symbol Device:Jumper_NO_Small
- added R15, R16, R17, R18: R, Resistor_SMD:R_0402_1005Metric, symbol Device:R
- added U4: MCP73831-2-OT, Package_TO_SOT_SMD:SOT-23-5, symbol Battery_Management:MCP73831-2-OT
Connections:
- net +BATT: now also C15.2, C21.2, C8.2, U4.3 (VBAT)
- net GND: now also C15.1, C20.2, C21.1, C8.1, D1.1 (K), R15.2, R16.2, U4.2 (VSS)
- new net: R17.2, R18.2, U4.1 (STAT)
- new net: JP1.1, R15.1, U4.5 (PROG)
- new net: D2.1 (K), R18.1
- new net: D1.2 (A), R17.1
- new net: JP1.2, R16.1
- new net +5V: C20.1, D2.2 (A), U4.4 (VDD)
Changed lines of the file:
@@
 	6950 1800 7500 1800
-$Comp
-L Device:CP C7
-U 1 1 5DB40CD1
-P 7500 1650
-F 0 "C7" H 7382 1604 50  0000 R CNN
-F 1 "CP" H 7382 1695 50  0000 R CNN
-F 2 "Capacitor_SMD:CP_Elec_3x5.3" H 7538 1500 50  0001 C CNN
-F 3 "~" H 7500 1650 50  0001 C CNN
-	1    7500 1650
-	-1   0    0    1
-$EndComp
 $Comp
 L power:GND #PWR0129
@@
 	0    1    1    0
 $EndComp
-Connection ~ 7500 1800
 $Comp
 L power:+BATT #PWR0131
@@
 	6950 4550 7500 4550
 $Comp
-L Device:CP C8
-U 1 1 5DB48091
-P 7500 4400
-F 0 "C8" H 7382 4354 50  0000 R CNN
-F 1 "CP" H 7382 4445 50  0000 R CNN
-F 2 "Capacitor_SMD:CP_Elec_3x5.3" H 7538 4250 50  0001 C CNN
-F 3 "~" H 7500 4400 50  0001 C CNN
-	1    7500 4400
-	-1   0    0    1
-$EndComp
-$Comp
 L power:GND #PWR0137
 U 1 1 5DB48097
@@
 	0    1    1    0
 $EndComp
-Connection ~ 7500 4550
 $Comp
 L power:+BATT #PWR0139
@@
 	0    -1   -1   0
 $EndComp
+$Comp
+L Battery_Management:MCP73831-2-OT U4
+U 1 1 5DB2A010
+P 9700 4800
+F 0 "U4" H 9300 5150 50  0000 C CNN
+F 1 "MCP73831-2-OT" H 9250 5050 50  0000 C CNN
+F 2 "Package_TO_SOT_SMD:SOT-23-5" H 9750 4550 50  0001 L CIN
+F 3 "http://ww1.microchip.com/downloads/en/DeviceDoc/20001984g.pdf" H 9550 4750 50  0001 C CNN
+	1    9700 4800
+	1    0    0    -1
+$EndComp
+Wire Wire Line
+	10100 4900 10300 4900
+$Comp
+L Device:R R18
+U 1 1 5DB2ACB5
+P 10450 4900
+F 0 "R18" V 10243 4900 50  0000 C CNN
+F 1 "R" V 10334 4900 50  0000 C CNN
+F 2 "Resistor_SMD:R_0402_1005Metric" V 10380 4900 50  0001 C CNN
+F 3 "~" H 10450 4900 50  0001 C CNN
+	1    10450 4900
+	0    1    1    0
+$EndComp
+$Comp
+L Device:LED D2
+U 1 1 5DB2BA71
+P 10750 4900
+F 0 "D2" H 10743 5116 50  0000 C CNN
+F 1 "LED" H 10743 5025 50  0000 C CNN
+F 2 "LED_SMD:LED_0603_1608Metric" H 10750 4900 50  0001 C CNN
+F 3 "~" H 10750 4900 50  0001 C CNN
+	1    10750 4900
+	1    0    0    -1
+$EndComp
+$Comp
+L power:+5V #PWR0169
+U 1 1 5DB2C28F
+P 10900 4900
+F 0 "#PWR0169" H 10900 4750 50  0001 C CNN
+F 1 "+5V" V 10915 5028 50  0000 L CNN
+F 2 "" H 10900 4900 50  0001 C CNN
+F 3 "" H 10900 4900 50  0001 C CNN
+	1    10900 4900
+	0    1    1    0
+$EndComp
+Wire Wire Line
+	10100 4900 10100 5150
+Wire Wire Line
+	10100 5150 10200 5150
+Connection ~ 10100 4900
+$Comp
+L Device:R R17
+U 1 1 5DB2CD6A
+P 10350 5150
+F 0 "R17" V 10143 5150 50  0000 C CNN
+F 1 "R" V 10234 5150 50  0000 C CNN
+F 2 "Resistor_SMD:R_0402_1005Metric" V 10280 5150 50  0001 C CNN
+F 3 "~" H 10350 5150 50  0001 C CNN
+	1    10350 5150
+	0    1    1    0
+$EndComp
+$Comp
+L Device:LED D1
+U 1 1 5DB2DA34
+P 10650 5150
+F 0 "D1" H 10643 4895 50  0000 C CNN
+F 1 "LED" H 10643 4986 50  0000 C CNN
+F 2 "LED_SMD:LED_0603_1608Metric" H 10650 5150 50  0001 C CNN
+F 3 "~" H 10650 5150 50  0001 C CNN
+	1    10650 5150
+	-1   0    0    1
+$EndComp
+$Comp
+L power:GND #PWR0170
+U 1 1 5DB2E3BF
+P 10800 5150
+F 0 "#PWR0170" H 10800 4900 50  0001 C CNN
+F 1 "GND" H 10805 4977 50  0000 C CNN
+F 2 "" H 10800 5150 50  0001 C CNN
+F 3 "" H 10800 5150 50  0001 C CNN
+	1    10800 5150
+	1    0    0    -1
+$EndComp
+$Comp
+L Device:C C21
+U 1 1 5DB2EACD
+P 10100 4550
+F 0 "C21" H 10215 4596 50  0000 L CNN
+F 1 "C" H 10215 4505 50  0000 L CNN
+F 2 "Capacitor_SMD:C_0402_1005Metric" H 10138 4400 50  0001 C CNN
+F 3 "~" H 10100 4550 50  0001 C CNN
+	1    10100 4550
+	1    0    0    -1
+$EndComp
+$Comp
+L power:+BATT #PWR0171
+U 1 1 5DB2F3F5
+P 10100 4700
+F 0 "#PWR0171" H 10100 4550 50  0001 C CNN
+F 1 "+BATT" V 10115 4828 50  0000 L CNN
+F 2 "" H 10100 4700 50  0001 C CNN
+F 3 "" H 10100 4700 50  0001 C CNN
+	1    10100 4700
+	0    1    1    0
+$EndComp
+Connection ~ 10100 4700
+$Comp
+L power:GND #PWR0172
+U 1 1 5DB2FC7E
+P 10100 4400
+F 0 "#PWR0172" H 10100 4150 50  0001 C CNN
+F 1 "GND" H 10105 4227 50  0000 C CNN
+F 2 "" H 10100 4400 50  0001 C CNN
+F 3 "" H 10100 4400 50  0001 C CNN
+	1    10100 4400
+	-1   0    0    1
+$EndComp
+Wire Wire Line
+	9700 4500 9700 4050
+$Comp
+L Device:C C20
+U 1 1 5DB30775
+P 9550 4050
+F 0 "C20" V 9298 4050 50  0000 C CNN
+F 1 "C" V 9389 4050 50  0000 C CNN
+F 2 "Capacitor_SMD:C_0402_1005Metric" H 9588 3900 50  0001 C CNN
+F 3 "~" H 9550 4050 50  0001 C CNN
+	1    9550 4050
+	0    1    1    0
+$EndComp
+$Comp
+L power:+5V #PWR0173
+U 1 1 5DB30FD0
+P 9700 4050
+F 0 "#PWR0173" H 9700 3900 50  0001 C CNN
+F 1 "+5V" H 9715 4223 50  0000 C CNN
+F 2 "" H 9700 4050 50  0001 C CNN
+F 3 "" H 9700 4050 50  0001 C CNN
+	1    9700 4050
+	1    0    0    -1
+$EndComp
+Connection ~ 9700 4050
+$Comp
+L power:GND #PWR0174
+U 1 1 5DB31616
+P 9400 4050
+F 0 "#PWR0174" H 9400 3800 50  0001 C CNN
+F 1 "GND" H 9405 3877 50  0000 C CNN
+F 2 "" H 9400 4050 50  0001 C CNN
+F 3 "" H 9400 4050 50  0001 C CNN
+	1    9400 4050
+	1    0    0    -1
+$EndComp
+Wire Wire Line
+	9300 4900 9200 4900
+$Comp
+L Device:R R15
+U 1 1 5DB321C4
+P 9050 4900
+F 0 "R15" V 8843 4900 50  0000 C CNN
+F 1 "R" V 8934 4900 50  0000 C CNN
+F 2 "Resistor_SMD:R_0402_1005Metric" V 8980 4900 50  0001 C CNN
+F 3 "~" H 9050 4900 50  0001 C CNN
+	1    9050 4900
+	0    1    1    0
+$EndComp
+$Comp
+L Device:R R16
+U 1 1 5DB3268B
+P 9050 5200
+F 0 "R16" V 8843 5200 50  0000 C CNN
+F 1 "R" V 8934 5200 50  0000 C CNN
+F 2 "Resistor_SMD:R_0402_1005Metric" V 8980 5200 50  0001 C CNN
+F 3 "~" H 9050 5200 50  0001 C CNN
+	1    9050 5200
+	0    1    1    0
+$EndComp
+$Comp
+L power:GND #PWR0175
+U 1 1 5DB32EED
+P 8900 5300
+F 0 "#PWR0175" H 8900 5050 50  0001 C CNN
+F 1 "GND" H 8905 5127 50  0000 C CNN
+F 2 "" H 8900 5300 50  0001 C CNN
+F 3 "" H 8900 5300 50  0001 C CNN
+	1    8900 5300
+	1    0    0    -1
+$EndComp
+Wire Wire Line
+	8900 5300 8900 5200
+Connection ~ 8900 5200
+Wire Wire Line
+	8900 5200 8900 4900
+$Comp
+L Device:Jumper_NO_Small JP1
+U 1 1 5DB34BFA
+P 9200 5100
+F 0 "JP1" V 9154 5148 50  0000 L CNN
+F 1 "Jumper_NO_Small" V 9245 5148 50  0000 L CNN
+F 2 "Jumper:SolderJumper-2_P1.3mm_Open_Pad1.0x1.5mm" H 9200 5100 50  0001 C CNN
+F 3 "~" H 9200 5100 50  0001 C CNN
+	1    9200 5100
+	0    1    1    0
+$EndComp
+Wire Wire Line
+	9200 5000 9200 4900
+Connection ~ 9200 4900
+$Comp
+L power:GND #PWR0176
+U 1 1 5DB358CA
+P 9700 5100
+F 0 "#PWR0176" H 9700 4850 50  0001 C CNN
+F 1 "GND" H 9705 4927 50  0000 C CNN
+F 2 "" H 9700 5100 50  0001 C CNN
+F 3 "" H 9700 5100 50  0001 C CNN
+	1    9700 5100
+	1    0    0    -1
+$EndComp
+$Comp
+L Device:C C8
+U 1 1 5DB298B3
+P 7500 1650
+F 0 "C8" H 7615 1696 50  0000 L CNN
+F 1 "C" H 7615 1605 50  0000 L CNN
+F 2 "Capacitor_SMD:C_0805_2012Metric" H 7538 1500 50  0001 C CNN
+F 3 "~" H 7500 1650 50  0001 C CNN
+	1    7500 1650
+	1    0    0    -1
+$EndComp
+Connection ~ 7500 1800
+$Comp
+L Device:C C15
+U 1 1 5DB29F98
+P 7500 4400
+F 0 "C15" H 7615 4446 50  0000 L CNN
+F 1 "C" H 7615 4355 50  0000 L CNN
+F 2 "Capacitor_SMD:C_0805_2012Metric" H 7538 4250 50  0001 C CNN
+F 3 "~" H 7500 4400 50  0001 C CNN
+	1    7500 4400
+	1    0    0    -1
+$EndComp
+Connection ~ 7500 4550
 $EndSCHEMATC
