File: SwarmBot.kicad_pcb (KiCad board)
At the start: 2 copper layers, 100.4 x 50.1 mm, 63 parts, among them IC1 ESP32-PICO-D4, IC2 A3916GESTR-T, IC3 A3916GESTR-T, IC4 A3916GESTR-T, J1 Conn_01x06_Female, J2 Conn_01x06_Female, J3 Conn_01x06_Female, J4 Conn_01x06_Female, J5 Conn_01x06_Female, J6 Conn_01x08_Female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

Commit message: correct according to cad
Parts:
- moved H9 2.78 mm to (5.61, 9.65)
- moved H10 2.76 mm to (17.6, 9.65)
Changed lines of the file:
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@@
-(kicad_pcb (version 20171130) (host pcbnew 5.1.4-e60b266~84~ubuntu18.04.1)
+(kicad_pcb (version 20171130) (host pcbnew "(5.0.0-rc3-dev-11-geaf938c7e)")
   (general
     (thickness 1.6)
@@
     (zone_45_only no)
     (trace_min 0.2)
+    (segment_width 0.2)
+    (edge_width 0.05)
     (via_size 0.8)
     (via_drill 0.4)
@@
     (uvia_min_size 0.2)
     (uvia_min_drill 0.1)
-    (edge_width 0.05)
-    (segment_width 0.2)
     (pcb_text_width 0.3)
     (pcb_text_size 1.5 1.5)
@@
     (solder_mask_min_width 0.25)
     (aux_axis_origin 0 0)
-    (visible_elements FFFFF77F)
+    (visible_elements 7FFFFFFF)
     (pcbplotparams
       (layerselection 0x010fc_ffffffff)
@@
     (add_net +5V)
     (add_net +BATT)
-    (add_net /Sheet5DAF9EB0/A1_2)
-    (add_net /Sheet5DAF9EB0/A2_2)
-    (add_net /Sheet5DAF9EB0/B1_2)
-    (add_net /Sheet5DAF9EB0/B2_2)
-    (add_net /Sheet5DAF9EB0/CKI)
     (add_net /Sheet5DAF9EB0/DTR)
     (add_net /Sheet5DAF9EB0/D_N)
@@
     (add_net /Sheet5DAF9EB0/SCL)
     (add_net /Sheet5DAF9EB0/SDA)
-    (add_net /Sheet5DAF9EB0/SDI)
     (add_net /Sheet5DAF9EB0/TX)
     (add_net /Sheet5DAF9EF1/A1)
@@
     (add_net "Net-(C16-Pad1)")
     (add_net "Net-(C2-Pad2)")
-    (add_net "Net-(IC1-Pad10)")
-    (add_net "Net-(IC1-Pad11)")
-    (add_net "Net-(IC1-Pad12)")
-    (add_net "Net-(IC1-Pad13)")
-    (add_net "Net-(IC1-Pad24)")
-    (add_net "Net-(IC1-Pad25)")
-    (add_net "Net-(IC1-Pad26)")
-    (add_net "Net-(IC1-Pad27)")
-    (add_net "Net-(IC1-Pad28)")
-    (add_net "Net-(IC1-Pad29)")
-    (add_net "Net-(IC1-Pad30)")
-    (add_net "Net-(IC1-Pad31)")
-    (add_net "Net-(IC1-Pad32)")
-    (add_net "Net-(IC1-Pad33)")
-    (add_net "Net-(IC1-Pad34)")
-    (add_net "Net-(IC1-Pad36)")
-    (add_net "Net-(IC1-Pad44)")
-    (add_net "Net-(IC1-Pad45)")
-    (add_net "Net-(IC1-Pad47)")
-    (add_net "Net-(IC1-Pad48)")
-    (add_net "Net-(IC1-Pad5)")
-    (add_net "Net-(IC1-Pad6)")
-    (add_net "Net-(IC1-Pad7)")
-    (add_net "Net-(IC1-Pad8)")
     (add_net "Net-(IC2-Pad13)")
-    (add_net "Net-(IC2-Pad16)")
-    (add_net "Net-(IC2-Pad7)")
     (add_net "Net-(IC2-Pad9)")
     (add_net "Net-(IC3-Pad13)")
-    (add_net "Net-(IC3-Pad16)")
-    (add_net "Net-(IC3-Pad7)")
     (add_net "Net-(IC3-Pad9)")
     (add_net "Net-(IC4-Pad13)")
-    (add_net "Net-(IC4-Pad16)")
-    (add_net "Net-(IC4-Pad7)")
     (add_net "Net-(IC4-Pad9)")
-    (add_net "Net-(J7-Pad4)")
     (add_net "Net-(Q1-Pad1)")
     (add_net "Net-(Q2-Pad1)")
     (add_net "Net-(R11-Pad1)")
-    (add_net "Net-(U1-Pad4)")
-    (add_net "Net-(U2-Pad10)")
-    (add_net "Net-(U2-Pad11)")
-    (add_net "Net-(U2-Pad12)")
-    (add_net "Net-(U2-Pad4)")
-    (add_net "Net-(U2-Pad9)")
-    (add_net "Net-(U3-Pad1)")
-    (add_net "Net-(U3-Pad10)")
-    (add_net "Net-(U3-Pad11)")
-    (add_net "Net-(U3-Pad12)")
-    (add_net "Net-(U3-Pad13)")
-    (add_net "Net-(U3-Pad14)")
-    (add_net "Net-(U3-Pad15)")
-    (add_net "Net-(U3-Pad16)")
-    (add_net "Net-(U3-Pad17)")
-    (add_net "Net-(U3-Pad18)")
-    (add_net "Net-(U3-Pad22)")
-    (add_net "Net-(U3-Pad24)")
-    (add_net "Net-(U3-Pad9)")
   )
   (module Package_DFN_QFN:QFN-24-1EP_4x4mm_P0.5mm_EP2.6x2.6mm (layer F.Cu)
@@
   )
   (module MountingHole:MountingHole_2.5mm (layer F.Cu)
-    (at 16.8529 12.3063)
+    (at 17.61 9.65)
     (descr "Mounting Hole 2.5mm, no annular")
     (tags "mounting hole 2.5mm no annular")
@@
   )
   (module MountingHole:MountingHole_2.5mm (layer F.Cu)
-    (at 6.44144 12.3063)
+    (at 5.61 9.65)
     (descr "Mounting Hole 2.5mm, no annular")
     (tags "mounting hole 2.5mm no annular")

Commit message: routed and reshaped
Parts:
- added C20: C, Capacitor_SMD:C_0402_1005Metric, F.Cu at (41.6, -11.9)
- added C21: C, Capacitor_SMD:C_0402_1005Metric, F.Cu at (38.5, -13.6)
- added D1: LED, LED_SMD:LED_0603_1608Metric, F.Cu at (40.7, -17.0)
- added D2: LED, LED_SMD:LED_0603_1608Metric, F.Cu at (36.6, -17.4)
- added J8: Conn_01x02_Male, Connector_JST:JST_PH_B2B-PH-K_1x02_P2.00mm_Vertical, F.Cu at (10.0, -16.4)
- added JP1: Jumper_NO_Small, Jumper:SolderJumper-2_P1.3mm_Open_Pad1.0x1.5mm, F.Cu at (44.3, -15.9)
- added R15: R, Resistor_SMD:R_0402_1005Metric, F.Cu at (46.6, -15.2)
- added R16: R, Resistor_SMD:R_0402_1005Metric, F.Cu at (43.8, -18.1)
- added R17: R, Resistor_SMD:R_0402_1005Metric, F.Cu at (38.6, -15.8)
- added R18: R, Resistor_SMD:R_0402_1005Metric, F.Cu at (37.1, -15.3)
- added U4: MCP73831-2-OT, Package_TO_SOT_SMD:SOT-23-5, F.Cu at (41.1, -14.3)
- C15, C7, C8: value CP -> C; footprint Capacitor_SMD:CP_Elec_3x5.3 -> Capacitor_SMD:C_0805_2012Metric
- J1: value Conn_01x06_Female -> Conn_01x04_Female; footprint Connector_PinHeader_2.00mm:PinHeader_1x06_P2.00mm_Vertical -> Connector_PinHeader_1.27mm:PinHeader_1x04_P1.27mm_Vertical
- J7: footprint Connector_USB:USB_Micro-B_Molex-105017-0001 -> Connector_USB:USB_Micro-B_Molex_47346-0001
- moved C15 61.7 mm to (28.4, -5.09), turned to 270 degrees
- moved R9 58.8 mm to (10.3, 20.3), turned to 180 degrees
- moved C14 58.3 mm to (9.86, 18.4), turned to 180 degrees
- moved IC4 58.1 mm to (6.42, 19.5)
- moved R8 57.2 mm to (8.15, 16.1), turned to 180 degrees
- moved C5 53.6 mm to (66.1, 15.1)
- moved IC2 53.6 mm to (64.9, 12.3)
- moved R1 53.6 mm to (63.6, 16.2)
- moved R3 53.6 mm to (61.7, 10.1)
- moved R10 48.1 mm to (-0.32, 13.8), turned to 270 degrees
- moved J1 45.8 mm to (10.7, 8.45), turned to 90 degrees
- moved C8 42.5 mm to (22.9, 5.42), turned to 90 degrees
- moved C16 40.7 mm to (-16.4, 10.3), turned to 90 degrees
- moved Q1 39.3 mm to (-15.2, -6.59), turned to 90 degrees
- moved C18 37.7 mm to (-15.3, 3.63), turned to 270 degrees
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Connections:
- C15 pad 1: +BATT -> GND
- C15 pad 2: GND -> +BATT
- C7 pad 1: +BATT -> GND
- C7 pad 2: GND -> +BATT
- C8 pad 1: +BATT -> GND
- C8 pad 2: GND -> +BATT
- IC1 pad 12: (no net) -> /Sheet5DAF9EB0/M2B_3
- IC1 pad 13: (no net) -> /Sheet5DAF9EB0/M2A_3
- IC1 pad 14: /Sheet5DAF9EB0/M2A_2 -> /Sheet5DAF9EB0/M1A_3
- IC1 pad 15: /Sheet5DAF9EB0/M2B_2 -> /Sheet5DAF9EB0/M1B_3
- IC1 pad 16: /Sheet5DAF9EB0/M1A_2 -> (no net)
- IC1 pad 17: /Sheet5DAF9EB0/M1B_2 -> (no net)
- IC1 pad 18: /Sheet5DAF9EB0/M2B -> /Sheet5DAF9EB0/M1B
- IC1 pad 20: /Sheet5DAF9EB0/M2A -> /Sheet5DAF9EB0/M1A
- IC1 pad 21: /Sheet5DAF9EB0/M1B -> /Sheet5DAF9EB0/M2B
- IC1 pad 22: /Sheet5DAF9EB0/M1A -> /Sheet5DAF9EB0/M2A
- IC1 pad 24: (no net) -> /Sheet5DAF9EB0/M2B_2
- IC1 pad 25: (no net) -> /Sheet5DAF9EB0/M1B_2
- IC1 pad 27: (no net) -> /Sheet5DAF9EB0/M2A_2
- IC1 pad 34: (no net) -> /Sheet5DAF9EB0/M1A_2
- IC4 pad 10: (no net) -> /Sheet5DAF9EB0/B2_3
- IC4 pad 12: (no net) -> /Sheet5DAF9EB0/B1_3
- IC4 pad 14: (no net) -> /Sheet5DAF9EB0/A1_3
- IC4 pad 3: /Sheet5DAF9EB0/M1A_2 -> /Sheet5DAF9EB0/M1A_3
- IC4 pad 4: /Sheet5DAF9EB0/M1B_2 -> /Sheet5DAF9EB0/M1B_3
- IC4 pad 5: /Sheet5DAF9EB0/M2A_2 -> /Sheet5DAF9EB0/M2A_3
- IC4 pad 6: /Sheet5DAF9EB0/M2B_2 -> /Sheet5DAF9EB0/M2B_3
- IC4 pad 8: (no net) -> /Sheet5DAF9EB0/A2_3
- J1 pad 1: +3V3 -> /Sheet5DAF9EB0/A1_3
- J1 pad 2: /Sheet5DAF9EB0/RX -> /Sheet5DAF9EB0/B1_3
- J1 pad 3: /Sheet5DAF9EB0/TX -> /Sheet5DAF9EB0/B2_3
- J1 pad 4: GND -> /Sheet5DAF9EB0/A2_3
- R10 pad 1: /Sheet5DAF9EB0/M2B -> /Sheet5DAF9EB0/M1B
Routing:
- net GND: track 0.00 -> 81.5 mm, vias 0 -> 128
- net /Sheet5DAF9EB0/IO0: track 0.00 -> 36.7 mm, vias 0 -> 4
- net /Sheet5DAF9EB0/EN: track 0.00 -> 35.9 mm, vias 0 -> 4
- net /Sheet5DAF9EB0/SDA: track 0.00 -> 31.4 mm, vias 0 -> 2
- net /Sheet5DAF9EB0/M1A: track 0.00 -> 29.4 mm, vias 0 -> 3
- net +5V: track 0.00 -> 28.4 mm, vias 0 -> 16
- net /Sheet5DAF9EB0/SCL: track 0.00 -> 27.4 mm, vias 0 -> 2
- net /Sheet5DAF9EB0/M1B: track 0.00 -> 26.6 mm, vias 0 -> 3
- net /Sheet5DAF9EF1/M2B_2: track 0.00 -> 25.9 mm, vias 0 -> 2
- net /Sheet5DAF9EB0/M2A: track 0.00 -> 24.8 mm, vias 0 -> 1
- net /Sheet5DAF9EF1/M1B_2: track 0.00 -> 24.1 mm, vias 0 -> 2
- net /Sheet5DAF9EB0/TX: track 0.00 -> 22.8 mm, vias 0 -> 4
- net /Sheet5DAF9EF1/M2A_2: track 0.00 -> 22.5 mm, vias 0 -> 2
- net /Sheet5DAF9EF1/M1A_2: track 0.00 -> 22.0 mm
- net /Sheet5DAF9EB0/M2B: track 0.00 -> 21.7 mm, vias 0 -> 1
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- added copper zone on B.Cu, net +5V
- added copper zone on B.Cu, net +BATT
Other:
- board size 100.4 x 50.1 mm -> 98.3 x 50 mm
