File: TopBoard.sch (KiCad schematic (older format))
At the start: 43 parts, among them IC1 ESP32-PICO-D4, IC4 A3916GESTR-T, J2 Conn_01x06_Female, J3 Conn_01x06_Female, J7 USB_B_Micro, Q1 MMBT3904, Q2 MMBT3904, SW1 SW_Push_Open, SW2 SW_Push_Open, U1 MIC5366-3.3YC5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

Commit message: routed and reshaped
Parts:
- removed C15: CP, Capacitor_SMD:CP_Elec_3x5.3, symbol Device:CP
- added C7: C, Capacitor_SMD:C_0805_2012Metric, symbol Device:C
- added J1: Conn_01x04_Female, Connector_PinHeader_1.27mm:PinHeader_1x04_P1.27mm_Vertical, symbol Connector:Conn_01x04_Female
- added J8: Conn_01x02_Male, Connector_JST:JST_PH_B2B-PH-K_1x02_P2.00mm_Vertical, symbol Connector:Conn_01x02_Male
- J7: footprint Connector_USB:USB_Micro-B_Molex-105017-0001 -> Connector_USB:USB_Micro-B_Molex_47346-0001
Connections:
- net +BATT: now also C7.2, J8.2 (Pin_2)
- net GND: now also C7.1, J8.1 (Pin_1)
- net M1A: now also IC1.20 (IO13); no longer IC1.22 (IO2)
- net M1A_2: now also IC1.34 (IO5); no longer IC1.16 (IO27), IC4.3 (IN1)
- net M1B: now also IC1.18 (IO12), R10.1; no longer IC1.21 (IO15)
- net M1B_2: now also IC1.25 (IO16); no longer IC1.17 (IO14), IC4.4 (IN2)
- net M2A: now also IC1.22 (IO2); no longer IC1.20 (IO13)
- net M2A_2: now also IC1.27 (IO17); no longer IC1.14 (IO25), IC4.5 (IN3)
- net M2B: now also IC1.21 (IO15); no longer IC1.18 (IO12), R10.1
- net M2B_2: now also IC1.24 (IO4); no longer IC1.15 (IO26), IC4.6 (IN4)
- net M2B_3: now reaches IC1.12 (IO32)
- net M2B_3: now also IC4.6 (IN4)
- net M2A_3: now reaches IC1.13 (IO33)
- net M2A_3: now also IC4.5 (IN3)
- net A1_2 renamed A1_3
- net A1_3: now also J1.1 (Pin_1)
- net A2_2 renamed A2_3
- net A2_3: now also J1.4 (Pin_4)
- net B1_2 renamed B1_3
- net B1_3: now also J1.2 (Pin_2)
- net B2_2 renamed B2_3
- net B2_3: now also J1.3 (Pin_3)
- net CKI: no longer names the net of IC1.35 (IO18)
- new net M1A_3: IC1.14 (IO25), IC4.3 (IN1)
- new net M1B_3: IC1.15 (IO26), IC4.4 (IN2)
- no-connect marks 17 -> 31
Changed lines of the file:
@@
 	-1   0    0    1
 $EndComp
+Text Label 2250 3400 2    50   ~ 0
+M1A
+Text Label 1800 3300 2    50   ~ 0
+M1B
 Text Label 2250 3600 2    50   ~ 0
-M1A
+M2A
 Text Label 2250 3500 2    50   ~ 0
-M1B
-Text Label 2250 3400 2    50   ~ 0
-M2A
-Text Label 1800 3300 2    50   ~ 0
 M2B
-Text Label 2250 3100 2    50   ~ 0
+Text Label 4050 2900 0    50   ~ 0
 M1A_2
-Text Label 2250 3200 2    50   ~ 0
+Text Label 2250 3900 2    50   ~ 0
 M1B_2
-Text Label 2250 2900 2    50   ~ 0
+Text Label 2250 4100 2    50   ~ 0
 M2A_2
-Text Label 2250 3000 2    50   ~ 0
+Text Label 2250 3800 2    50   ~ 0
 M2B_2
 $Comp
@@
 $EndComp
 Connection ~ 9600 3250
-Text Label 4050 3000 0    50   ~ 0
-CKI
 Text Label 4050 3300 0    50   ~ 0
 SDI
@@
 $EndComp
 Text Label 5600 5450 1    50   ~ 0
-A1_2
+A1_3
 Text Label 5600 7150 3    50   ~ 0
-A2_2
+A2_3
 Text Label 6200 6150 0    50   ~ 0
-B1_2
+B1_3
 Text Label 6200 6350 0    50   ~ 0
-B2_2
+B2_3
 $Comp
 L power:GND #PWR?
@@
 $EndComp
 Text Label 4800 6350 2    50   ~ 0
-M1A_2
+M1A_3
 Text Label 4800 6450 2    50   ~ 0
-M1B_2
+M1B_3
 Text Label 5300 7150 3    50   ~ 0
-M2A_2
+M2A_3
 Text Label 5400 7150 3    50   ~ 0
-M2B_2
+M2B_3
 $Comp
 L Device:R R?
@@
 	6200 6250 6750 6250
 $Comp
-L Device:CP C?
-U 1 1 5DB307E7
-P 6750 6100
-AR Path="/5DAF9EF2/5DB307E7" Ref="C?"  Part="1"
-AR Path="/5DAF9EB1/5DB307E7" Ref="C15"  Part="1"
-F 0 "C15" H 6632 6054 50  0000 R CNN
-F 1 "CP" H 6632 6145 50  0000 R CNN
-F 2 "Capacitor_SMD:CP_Elec_3x5.3" H 6788 5950 50  0001 C CNN
-F 3 "~" H 6750 6100 50  0001 C CNN
-	1    6750 6100
-	-1   0    0    1
-$EndComp
-$Comp
 L power:GND #PWR?
 U 1 1 5DB307ED
@@
 	0    1    1    0
 $EndComp
-Connection ~ 6750 6250
 $Comp
 L power:+BATT #PWR?
@@
 F 0 "J7" H 5057 2367 50  0000 C CNN
 F 1 "USB_B_Micro" H 5057 2276 50  0000 C CNN
-F 2 "Connector_USB:USB_Micro-B_Molex-105017-0001" H 5150 1850 50  0001 C CNN
+F 2 "Connector_USB:USB_Micro-B_Molex_47346-0001" H 5150 1850 50  0001 C CNN
 F 3 "~" H 5150 1850 50  0001 C CNN
 	1    5000 1900
@@
 	1    0    0    -1
 $EndComp
+$Comp
+L Device:C C7
+U 1 1 5DB284B9
+P 6750 6100
+F 0 "C7" H 6865 6146 50  0000 L CNN
+F 1 "C" H 6865 6055 50  0000 L CNN
+F 2 "Capacitor_SMD:C_0805_2012Metric" H 6788 5950 50  0001 C CNN
+F 3 "~" H 6750 6100 50  0001 C CNN
+	1    6750 6100
+	1    0    0    -1
+$EndComp
+Connection ~ 6750 6250
+$Comp
+L Connector:Conn_01x02_Male J8
+U 1 1 5DB46B22
+P 7350 3900
+F 0 "J8" V 7412 3944 50  0000 L CNN
+F 1 "Conn_01x02_Male" V 7503 3944 50  0000 L CNN
+F 2 "Connector_JST:JST_PH_B2B-PH-K_1x02_P2.00mm_Vertical" H 7350 3900 50  0001 C CNN
+F 3 "~" H 7350 3900 50  0001 C CNN
+	1    7350 3900
+	0    1    1    0
+$EndComp
+$Comp
+L power:+BATT #PWR0177
+U 1 1 5DB4816C
+P 7250 4100
+F 0 "#PWR0177" H 7250 3950 50  0001 C CNN
+F 1 "+BATT" H 7265 4273 50  0000 C CNN
+F 2 "" H 7250 4100 50  0001 C CNN
+F 3 "" H 7250 4100 50  0001 C CNN
+	1    7250 4100
+	-1   0    0    1
+$EndComp
+Wire Wire Line
+	7350 4100 7350 4350
+$Comp
+L power:GND #PWR0178
+U 1 1 5DB4AFA6
+P 7350 4350
+F 0 "#PWR0178" H 7350 4100 50  0001 C CNN
+F 1 "GND" H 7355 4177 50  0000 C CNN
+F 2 "" H 7350 4350 50  0001 C CNN
+F 3 "" H 7350 4350 50  0001 C CNN
+	1    7350 4350
+	1    0    0    -1
+$EndComp
+$Comp
+L Connector:Conn_01x04_Female J1
+U 1 1 5DB3079D
+P 5600 3900
+F 0 "J1" V 5538 3612 50  0000 R CNN
+F 1 "Conn_01x04_Female" V 5447 3612 50  0000 R CNN
+F 2 "Connector_PinHeader_1.27mm:PinHeader_1x04_P1.27mm_Vertical" H 5600 3900 50  0001 C CNN
+F 3 "~" H 5600 3900 50  0001 C CNN
+	1    5600 3900
+	0    -1   -1   0
+$EndComp
+Text Label 5500 4100 3    50   ~ 0
+A1_3
+Text Label 5600 4100 3    50   ~ 0
+B1_3
+Text Label 5700 4100 3    50   ~ 0
+B2_3
+Text Label 5800 4100 3    50   ~ 0
+A2_3
+Text Label 2250 2900 2    50   ~ 0
+M1A_3
+Text Label 2250 3000 2    50   ~ 0
+M1B_3
+Text Label 2250 2800 2    50   ~ 0
+M2A_3
+Text Label 2250 2700 2    50   ~ 0
+M2B_3
+NoConn ~ 2250 4200
+NoConn ~ 2250 4300
+NoConn ~ 2250 4400
+NoConn ~ 2250 4500
+NoConn ~ 2250 4600
+NoConn ~ 2250 4700
+NoConn ~ 4050 3800
+NoConn ~ 4050 3900
+NoConn ~ 4050 4000
+NoConn ~ 4050 4100
+NoConn ~ 4050 4200
+NoConn ~ 4050 2800
+NoConn ~ 4050 2700
+NoConn ~ 4050 2600
 $EndSCHEMATC
